Commit message: urdf folder renamed to xacro folder. Description files translated to xacro language.

File: phantomx_description/xacro/robot_parameters.xacro (robot description, xacro)
@@ -1,4 +1,3 @@
 <?xml version="1.0" ?>
-<!-- values -->
 <robot xmlns:xacro="http://www.ros.org/wiki/xacro">
 	<!-- Link names -->
@@ -35,18 +34,18 @@
 	<xacro:property name="actr_04_name" value="finger_1_joint_motor" />
 	<xacro:property name="actr_05_name" value="finger_2_joint_motor" />
-	<!--  geometry mesh files  6-->
+	<!-- visual mesh files -->
 	<xacro:property name="geom_00_name" value="package://phantomx_description/models/phantomx_pincher/meshes/visual/base.dae" />
-	<xacro:property name="geom_01_name" value="package://phantomx_description/models/phantomx_pincher/meshes/visual/shoulder.dae"  />
+	<xacro:property name="geom_01_name" value="package://phantomx_description/models/phantomx_pincher/meshes/visual/shoulder.dae" />
 	<xacro:property name="geom_02_name" value="package://phantomx_description/models/phantomx_pincher/meshes/visual/lower_arm.dae" />
-	<xacro:property name="geom_03_name" value="package://phantomx_description/models/phantomx_pincher/meshes/visual/upper_arm.dae" />
+	<xacro:property name="geom_03_name" value="package://phantomx_description/models/phantomx_pincher/meshes/visual/lower_arm.dae" />
 	<xacro:property name="geom_04_name" value="package://phantomx_description/models/phantomx_pincher/meshes/visual/gripper_body.dae" />
 	<xacro:property name="geom_05_name" value="package://phantomx_description/models/phantomx_pincher/meshes/visual/finger.dae" />
 	<xacro:property name="geom_06_name" value="package://phantomx_description/models/phantomx_pincher/meshes/visual/finger.dae" />
-	<!-- collision mesh files  5-->
+	<!-- collision mesh files -->
 	<xacro:property name="colli_00_name" value="package://phantomx_description/models/phantomx_pincher/meshes/collision/simple_base.dae" />
 	<xacro:property name="colli_01_name" value="package://phantomx_description/models/phantomx_pincher/meshes/collision/simple_shoulder.dae" />
 	<xacro:property name="colli_02_name" value="package://phantomx_description/models/phantomx_pincher/meshes/collision/simple_bicep.dae" />
 	<xacro:property name="colli_03_name" value="package://phantomx_description/models/phantomx_pincher/meshes/collision/simple_bicep.dae" />
-	<xacro:property name="colli_04_name" value="package://phantomx_description/models/phantomx_pincher/meshes/collision/simple_wrist.dae"  />
+	<xacro:property name="colli_04_name" value="package://phantomx_description/models/phantomx_pincher/meshes/collision/simple_wrist.dae" />
 	<xacro:property name="colli_05_name" value="package://phantomx_description/models/phantomx_pincher/meshes/collision/simple_finger.dae" />
 	<xacro:property name="colli_06_name" value="package://phantomx_description/models/phantomx_pincher/meshes/collision/simple_finger.dae" />
